File: pcb/discrete/discrete-rf-board/lna_gain_block.sch (KiCad schematic (older format))
At the start: 20 parts

Commit message: Merge stuff I guess, hopefully this doesn't break too much
Parts:
- removed C?: 100 pF RF, symbol Device:C_Small
- removed Q?: Q_NPN_BCE, symbol Device:Q_NPN_BCE
- removed R?: 200R, symbol Device:R_Small
- added C?: 100 pF RF, symbol Device:C_Small
- added Q801: Q_NPN_BCEE, symbol discrete-parts:Q_NPN_BCEE
- C804: renamed from C?; value 5.0 pF RF -> 5.45 pF RF
- C809: renamed from C?; value 2.6 pF RF -> 3.0 pF RF
- L801: renamed from L?; value 8.5 nH -> 9.5 nH
- L803: renamed from L?; value 2.6 nH -> 10.0 nH
- R801: renamed from R?; value 3k3R -> 8k2R
- R802: renamed from R?; value 1k7R -> 1k8R
- R803: renamed from R?; value 10R -> 75R
- R804: renamed from R?; value 3.3R -> 22R
- gave numbers to parts that had none: 9
Connections:
- net GND: now also C?.2, Q801.3 (E), Q801.4 (C)
- net at R803.1: now also C?.1
- net at L801.2: now also Q801.1 (B); no longer R803.2
- net at L802.2, L803.1: now also R803.2, Q801.2 (C)
Other:
- note added: "TODO make sure the matching circuit values are\ncalculated for Vce=5V"
- note added: "Vbe=~~0.827V, ib=~~0.05mA, ic=5mA\nNF=1.5 dB, K=~~16dB"
- moved on the sheet: C1009, C1010, L1003, R1003
