File: pcb/discrete/discrete-rf-board/switchable-attenuator.sch (KiCad schematic (older format))
At the start: 11 parts

Commit message: Merge stuff I guess, hopefully this doesn't break too much
Parts:
- gave numbers to parts that had none: 11
