File: pcb/discrete/discrete-rf-board/if_amp.sch (KiCad schematic (older format))
At the start: 48 parts, among them Q23 NSVT65011MW6T1G, Q24 Q_NPN_BCE, Q25 NSVT65011MW6T1G, U10 NLAS4157DFT2G, U11 NLAS4157DFT2G, U8 NLAS4157DFT2G, U9 NLAS4157DFT2G

Commit message: Footprint some stuff
Parts:
- TP7: footprint (none) -> TestPoint:TestPoint_Pad_D1.0mm; Mouser (none) -> NoPart
Changed lines of the file:
@@
 AR Path="/5CA6B0AA/5CC4DFC2/5CC541C5" Ref="#PWR0154"  Part="1"
 AR Path="/5CA6B0AA/5CC9409A/5CC541C5" Ref="#PWR0177"  Part="1"
-F 0 "#PWR0177" H 3250 3100 50  0001 C CNN
+F 0 "#PWR0154" H 3250 3100 50  0001 C CNN
 F 1 "GND" H 3250 3200 50  0000 C CNN
 F 2 "" H 3250 3350 50  0001 C CNN
@@
 AR Path="/5CA6B0AA/5CC4DFC2/5CC543E7" Ref="#PWR0150"  Part="1"
 AR Path="/5CA6B0AA/5CC9409A/5CC543E7" Ref="#PWR0173"  Part="1"
-F 0 "#PWR0173" H 1650 3100 50  0001 C CNN
+F 0 "#PWR0150" H 1650 3100 50  0001 C CNN
 F 1 "GND" H 1650 3200 50  0000 C CNN
 F 2 "" H 1650 3350 50  0001 C CNN
@@
 AR Path="/5CA6B0AA/5CC4DFC2/5CC54945" Ref="#PWR0151"  Part="1"
 AR Path="/5CA6B0AA/5CC9409A/5CC54945" Ref="#PWR0174"  Part="1"
-F 0 "#PWR0174" H 2450 4050 50  0001 C CNN
+F 0 "#PWR0151" H 2450 4050 50  0001 C CNN
 F 1 "GND" H 2450 4150 50  0000 C CNN
 F 2 "" H 2450 4300 50  0001 C CNN
@@
 AR Path="/5CA6B0AA/5CC4DFC2/5CC64E30" Ref="#PWR0149"  Part="1"
 AR Path="/5CA6B0AA/5CC9409A/5CC64E30" Ref="#PWR0172"  Part="1"
-F 0 "#PWR0172" H 1300 3900 50  0001 C CNN
+F 0 "#PWR0149" H 1300 3900 50  0001 C CNN
 F 1 "GND" H 1300 4000 50  0000 C CNN
 F 2 "" H 1300 4150 50  0001 C CNN
@@
 AR Path="/5CA6B0AA/5CC4DFC2/5CC71057" Ref="#PWR0165"  Part="1"
 AR Path="/5CA6B0AA/5CC9409A/5CC71057" Ref="#PWR0188"  Part="1"
-F 0 "#PWR0188" H 7350 2850 50  0001 C CNN
+F 0 "#PWR0165" H 7350 2850 50  0001 C CNN
 F 1 "GND" H 7350 2950 50  0000 C CNN
 F 2 "" H 7350 3100 50  0001 C CNN
@@
 AR Path="/5CA6B0AA/5CC4DFC2/5CC7105D" Ref="#PWR0163"  Part="1"
 AR Path="/5CA6B0AA/5CC9409A/5CC7105D" Ref="#PWR0186"  Part="1"
-F 0 "#PWR0186" H 5750 2850 50  0001 C CNN
+F 0 "#PWR0163" H 5750 2850 50  0001 C CNN
 F 1 "GND" H 5750 2950 50  0000 C CNN
 F 2 "" H 5750 3100 50  0001 C CNN
@@
 AR Path="/5CA6B0AA/5CC4DFC2/5CC7911F" Ref="#PWR0164"  Part="1"
 AR Path="/5CA6B0AA/5CC9409A/5CC7911F" Ref="#PWR0187"  Part="1"
-F 0 "#PWR0187" H 6550 3650 50  0001 C CNN
+F 0 "#PWR0164" H 6550 3650 50  0001 C CNN
 F 1 "GND" H 6550 3750 50  0000 C CNN
 F 2 "" H 6550 3900 50  0001 C CNN
@@
 AR Path="/5CA6B0AA/5CC4DFC2/5CC9F407" Ref="#PWR0152"  Part="1"
 AR Path="/5CA6B0AA/5CC9409A/5CC9F407" Ref="#PWR0175"  Part="1"
-F 0 "#PWR0175" H 2500 6550 50  0001 C CNN
+F 0 "#PWR0152" H 2500 6550 50  0001 C CNN
 F 1 "GND" H 2500 6650 50  0000 C CNN
 F 2 "" H 2500 6800 50  0001 C CNN
@@
 AR Path="/5CA6B0AA/5CC4DFC2/5CC9FAC5" Ref="#PWR0155"  Part="1"
 AR Path="/5CA6B0AA/5CC9409A/5CC9FAC5" Ref="#PWR0178"  Part="1"
-F 0 "#PWR0178" H 3350 6550 50  0001 C CNN
+F 0 "#PWR0155" H 3350 6550 50  0001 C CNN
 F 1 "GND" H 3350 6650 50  0000 C CNN
 F 2 "" H 3350 6800 50  0001 C CNN
@@
 AR Path="/5CA6B0AA/5CC4DFC2/5CC9FD6D" Ref="#PWR0160"  Part="1"
 AR Path="/5CA6B0AA/5CC9409A/5CC9FD6D" Ref="#PWR0183"  Part="1"
-F 0 "#PWR0183" H 4300 6550 50  0001 C CNN
+F 0 "#PWR0160" H 4300 6550 50  0001 C CNN
 F 1 "GND" H 4300 6650 50  0000 C CNN
 F 2 "" H 4300 6800 50  0001 C CNN
@@
 AR Path="/5CA6B0AA/5CC4DFC2/5CCA0195" Ref="#PWR0162"  Part="1"
 AR Path="/5CA6B0AA/5CC9409A/5CCA0195" Ref="#PWR0185"  Part="1"
-F 0 "#PWR0185" H 5050 6550 50  0001 C CNN
+F 0 "#PWR0162" H 5050 6550 50  0001 C CNN
 F 1 "GND" H 5050 6650 50  0000 C CNN
 F 2 "" H 5050 6800 50  0001 C CNN
@@
 AR Path="/5CA6B0AA/5CC4DFC2/5CCA0420" Ref="#PWR0153"  Part="1"
 AR Path="/5CA6B0AA/5CC9409A/5CCA0420" Ref="#PWR0176"  Part="1"
-F 0 "#PWR0176" H 3050 5650 50  0001 C CNN
+F 0 "#PWR0153" H 3050 5650 50  0001 C CNN
 F 1 "GND" H 3050 5750 50  0000 C CNN
 F 2 "" H 3050 5900 50  0001 C CNN
@@
 AR Path="/5CA6B0AA/5CC4DFC2/5CCA07DE" Ref="#PWR0156"  Part="1"
 AR Path="/5CA6B0AA/5CC9409A/5CCA07DE" Ref="#PWR0179"  Part="1"
-F 0 "#PWR0179" H 3550 5650 50  0001 C CNN
+F 0 "#PWR0156" H 3550 5650 50  0001 C CNN
 F 1 "GND" H 3550 5750 50  0000 C CNN
 F 2 "" H 3550 5900 50  0001 C CNN
@@
 AR Path="/5CA6B0AA/5CC4DFC2/5CCA0A90" Ref="#PWR0158"  Part="1"
 AR Path="/5CA6B0AA/5CC9409A/5CCA0A90" Ref="#PWR0181"  Part="1"
-F 0 "#PWR0181" H 4000 5650 50  0001 C CNN
+F 0 "#PWR0158" H 4000 5650 50  0001 C CNN
 F 1 "GND" H 4000 5750 50  0000 C CNN
 F 2 "" H 4000 5900 50  0001 C CNN
@@
 AR Path="/5CA6B0AA/5CC4DFC2/5CCA0D69" Ref="#PWR0161"  Part="1"
 AR Path="/5CA6B0AA/5CC9409A/5CCA0D69" Ref="#PWR0184"  Part="1"
-F 0 "#PWR0184" H 4450 5650 50  0001 C CNN
+F 0 "#PWR0161" H 4450 5650 50  0001 C CNN
 F 1 "GND" H 4450 5750 50  0000 C CNN
 F 2 "" H 4450 5900 50  0001 C CNN
@@
 F 0 "TP7" H 5850 2420 50  0000 C CNN
 F 1 "TestPoint" H 5850 2350 50  0000 C CNN
-F 2 "" H 6050 2150 50  0001 C CNN
+F 2 "TestPoint:TestPoint_Pad_D1.0mm" H 6050 2150 50  0001 C CNN
 F 3 "~" H 6050 2150 50  0001 C CNN
+F 4 "NoPart" H 5850 2150 50  0001 C CNN "Mouser"
 	1    5850 2150
 	1    0    0    -1
@@
 AR Path="/5CA6B0AA/5CC4DFC2/5D57AB69" Ref="#PWR0157"  Part="1"
 AR Path="/5CA6B0AA/5CC9409A/5D57AB69" Ref="#PWR0180"  Part="1"
-F 0 "#PWR0180" H 3650 1900 50  0001 C CNN
+F 0 "#PWR0157" H 3650 1900 50  0001 C CNN
 F 1 "GND" H 3650 2000 50  0000 C CNN
 F 2 "" H 3650 2150 50  0001 C CNN
@@
 AR Path="/5CA6B0AA/5CC4DFC2/5D57AB6F" Ref="#PWR0159"  Part="1"
 AR Path="/5CA6B0AA/5CC9409A/5D57AB6F" Ref="#PWR0182"  Part="1"
-F 0 "#PWR0182" H 4100 1900 50  0001 C CNN
+F 0 "#PWR0159" H 4100 1900 50  0001 C CNN
 F 1 "GND" H 4100 2000 50  0000 C CNN
 F 2 "" H 4100 2150 50  0001 C CNN
@@
 AR Path="/5CA6B0AA/5CC4DFC2/5D580ADA" Ref="#PWR0166"  Part="1"
 AR Path="/5CA6B0AA/5CC9409A/5D580ADA" Ref="#PWR0189"  Part="1"
-F 0 "#PWR0189" H 7850 1650 50  0001 C CNN
+F 0 "#PWR0166" H 7850 1650 50  0001 C CNN
 F 1 "GND" H 7850 1750 50  0000 C CNN
 F 2 "" H 7850 1900 50  0001 C CNN
@@
 AR Path="/5CA6B0AA/5CC4DFC2/5D580AE0" Ref="#PWR0167"  Part="1"
 AR Path="/5CA6B0AA/5CC9409A/5D580AE0" Ref="#PWR0190"  Part="1"
-F 0 "#PWR0190" H 8300 1650 50  0001 C CNN
+F 0 "#PWR0167" H 8300 1650 50  0001 C CNN
 F 1 "GND" H 8300 1750 50  0000 C CNN
 F 2 "" H 8300 1900 50  0001 C CNN
