File: pcb/discrete/discrete-rf-board/if_amp.sch (KiCad schematic (older format))
At the start: 48 parts, among them Q15 NSVT65011MW6T1G, Q16 Q_NPN_BCE, Q17 NSVT65011MW6T1G, U10 NLAS4157DFT2G, U11 NLAS4157DFT2G, U8 NLAS4157DFT2G, U9 NLAS4157DFT2G

Commit message: Footprint a lot of stuff; save before autofill
Parts:
- C118: value 2.5 nF -> 2.2 nF; footprint (none) -> Capacitor_SMD:C_0402_1005Metric; Mouser (none) -> 81-GRM36X222K50
- R101, R99: value 25R -> 22R
- R108: footprint (none) -> Resistor_SMD:R_0402_1005Metric; Mouser (none) -> 603-RC0402JR-7D330RL
Changed lines of the file:
@@
 $Descr A4 11693 8268
 encoding utf-8
-Sheet 10 19
+Sheet 12 19
 Title ""
 Date ""
@@
 AR Path="/5CA6B0AA/5CC9409A/5CC4F99A" Ref="R125"  Part="1"
 F 0 "R125" H 2880 2270 50  0000 L CNN
-F 1 "25R" H 2880 2210 50  0000 L CNN
+F 1 "22R" H 2880 2210 50  0000 L CNN
 F 2 "" H 2850 2250 50  0001 C CNN
 F 3 "~" H 2850 2250 50  0001 C CNN
@@
 F 0 "R132" H 6580 3720 50  0000 L CNN
 F 1 "330R" H 6580 3660 50  0000 L CNN
-F 2 "" H 6550 3700 50  0001 C CNN
+F 2 "Resistor_SMD:R_0402_1005Metric" H 6550 3700 50  0001 C CNN
 F 3 "~" H 6550 3700 50  0001 C CNN
+F 4 "603-RC0402JR-7D330RL" H 6550 3700 50  0001 C CNN "Mouser"
 	1    6550 3700
 	1    0    0    -1
@@
 AR Path="/5CA6B0AA/5CC9409A/5DA03B3D" Ref="C142"  Part="1"
 F 0 "C142" H 2510 2520 50  0000 L CNN
-F 1 "2.5 nF" H 2510 2370 50  0000 L CNN
-F 2 "" H 2500 2450 50  0001 C CNN
+F 1 "2.2 nF" H 2510 2370 50  0000 L CNN
+F 2 "Capacitor_SMD:C_0402_1005Metric" H 2500 2450 50  0001 C CNN
 F 3 "~" H 2500 2450 50  0001 C CNN
+F 4 "81-GRM36X222K50" H 2500 2450 50  0001 C CNN "Mouser"
 	1    2500 2450
 	0    1    1    0
@@
 AR Path="/5CA6B0AA/5CC9409A/5CC4F475" Ref="R123"  Part="1"
 F 0 "R123" H 2080 2270 50  0000 L CNN
-F 1 "25R" H 2080 2210 50  0000 L CNN
+F 1 "22R" H 2080 2210 50  0000 L CNN
 F 2 "" H 2050 2250 50  0001 C CNN
 F 3 "~" H 2050 2250 50  0001 C CNN

Commit message: Autofill
Parts:
- R100, R101, R107, R110, R99: footprint (none) -> Resistor_SMD:R_0402_1005Metric; Mouser (none) -> 71-CRCW040222R0JNEDC
Changed lines of the file:
@@
 F 0 "R125" H 2880 2270 50  0000 L CNN
 F 1 "22R" H 2880 2210 50  0000 L CNN
-F 2 "" H 2850 2250 50  0001 C CNN
+F 2 "Resistor_SMD:R_0402_1005Metric" H 2850 2250 50  0001 C CNN
 F 3 "~" H 2850 2250 50  0001 C CNN
+F 4 "71-CRCW040222R0JNEDC" H 2850 2250 50  0001 C CNN "Mouser"
 	1    2850 2250
 	1    0    0    -1
@@
 F 0 "R124" H 2480 4120 50  0000 L CNN
 F 1 "22R" H 2480 4060 50  0000 L CNN
-F 2 "" H 2450 4100 50  0001 C CNN
+F 2 "Resistor_SMD:R_0402_1005Metric" H 2450 4100 50  0001 C CNN
 F 3 "~" H 2450 4100 50  0001 C CNN
+F 4 "71-CRCW040222R0JNEDC" H 2450 4100 50  0001 C CNN "Mouser"
 	1    2450 4100
 	1    0    0    -1
@@
 F 0 "R131" H 6180 3220 50  0000 L CNN
 F 1 "22R" H 6180 3160 50  0000 L CNN
-F 2 "" H 6150 3200 50  0001 C CNN
+F 2 "Resistor_SMD:R_0402_1005Metric" H 6150 3200 50  0001 C CNN
 F 3 "~" H 6150 3200 50  0001 C CNN
+F 4 "71-CRCW040222R0JNEDC" H 6150 3200 50  0001 C CNN "Mouser"
 	1    6150 3200
 	1    0    0    -1
@@
 F 0 "R134" H 6980 3170 50  0000 L CNN
 F 1 "22R" H 6980 3110 50  0000 L CNN
-F 2 "" H 6950 3150 50  0001 C CNN
+F 2 "Resistor_SMD:R_0402_1005Metric" H 6950 3150 50  0001 C CNN
 F 3 "~" H 6950 3150 50  0001 C CNN
+F 4 "71-CRCW040222R0JNEDC" H 6950 3150 50  0001 C CNN "Mouser"
 	1    6950 3150
 	1    0    0    -1
@@
 F 0 "R123" H 2080 2270 50  0000 L CNN
 F 1 "22R" H 2080 2210 50  0000 L CNN
-F 2 "" H 2050 2250 50  0001 C CNN
+F 2 "Resistor_SMD:R_0402_1005Metric" H 2050 2250 50  0001 C CNN
 F 3 "~" H 2050 2250 50  0001 C CNN
+F 4 "71-CRCW040222R0JNEDC" H 2050 2250 50  0001 C CNN "Mouser"
 	1    2050 2250
 	1    0    0    -1

Commit message: Autofill
Parts:
- C127: footprint (none) -> Capacitor_SMD:C_0402_1005Metric; Mouser (none) -> 81-GCM155R71H471K37D
Changed lines of the file:
@@
 F 0 "C151" H 6610 2270 50  0000 L CNN
 F 1 "470 pF" H 6610 2120 50  0000 L CNN
-F 2 "" H 6600 2200 50  0001 C CNN
+F 2 "Capacitor_SMD:C_0402_1005Metric" H 6600 2200 50  0001 C CNN
 F 3 "~" H 6600 2200 50  0001 C CNN
+F 4 "81-GCM155R71H471K37D" H 6600 2200 50  0001 C CNN "Mouser"
 	1    6600 2200
 	0    1    1    0
