File: pcb/discrete/discrete-rf-board/discrete-rf-board.sch (KiCad schematic (older format))
At the start: 22 parts, among them J1 Conn_01x11, J2 Conn_01x26, J3 Conn_01x30, J4 UFL, J5 UFL, J6 SMA, U1 BGS12PL6E6327XTSA1, U2 BGS12PL6E6327XTSA1

Commit message: Autofill
Parts:
- C1, C10, C11, C2: footprint (none) -> Capacitor_SMD:C_0402_1005Metric; Mouser (none) -> 791-RF15N101J250CT
- R2: footprint (none) -> Capacitor_SMD:C_0402_1005Metric; Mouser (none) -> 71-CRCW04020000Z0EDC
Changed lines of the file:
@@
 F 0 "R2" H 9780 3270 50  0000 L CNN
 F 1 "0R" H 9780 3210 50  0000 L CNN
-F 2 "" H 9750 3250 50  0001 C CNN
+F 2 "Capacitor_SMD:C_0402_1005Metric" H 9750 3250 50  0001 C CNN
 F 3 "~" H 9750 3250 50  0001 C CNN
+F 4 "71-CRCW04020000Z0EDC" H 9750 3250 50  0001 C CNN "Mouser"
 	1    9750 3250
 	0    -1   -1   0
@@
 F 0 "C2" H 2910 2170 50  0000 L CNN
 F 1 "100 pF" H 2910 2020 50  0000 L CNN
-F 2 "" H 2900 2100 50  0001 C CNN
+F 2 "Capacitor_SMD:C_0402_1005Metric" H 2900 2100 50  0001 C CNN
 F 3 "~" H 2900 2100 50  0001 C CNN
+F 4 "791-RF15N101J250CT " H 2900 2100 50  0001 C CNN "Mouser"
 	1    2900 2100
 	1    0    0    -1
@@
 F 0 "C1" H 2560 2170 50  0000 L CNN
 F 1 "100 pF" H 2560 2020 50  0000 L CNN
-F 2 "" H 2550 2100 50  0001 C CNN
+F 2 "Capacitor_SMD:C_0402_1005Metric" H 2550 2100 50  0001 C CNN
 F 3 "~" H 2550 2100 50  0001 C CNN
+F 4 "791-RF15N101J250CT " H 2550 2100 50  0001 C CNN "Mouser"
 	1    2550 2100
 	1    0    0    -1
@@
 F 0 "C10" H 9810 2370 50  0000 L CNN
 F 1 "100 pF" H 9810 2220 50  0000 L CNN
-F 2 "" H 9800 2300 50  0001 C CNN
+F 2 "Capacitor_SMD:C_0402_1005Metric" H 9800 2300 50  0001 C CNN
 F 3 "~" H 9800 2300 50  0001 C CNN
+F 4 "791-RF15N101J250CT " H 9800 2300 50  0001 C CNN "Mouser"
 	1    9800 2300
 	-1   0    0    -1
@@
 F 0 "C11" H 10160 2370 50  0000 L CNN
 F 1 "100 pF" H 10160 2220 50  0000 L CNN
-F 2 "" H 10150 2300 50  0001 C CNN
+F 2 "Capacitor_SMD:C_0402_1005Metric" H 10150 2300 50  0001 C CNN
 F 3 "~" H 10150 2300 50  0001 C CNN
+F 4 "791-RF15N101J250CT " H 10150 2300 50  0001 C CNN "Mouser"
 	1    10150 2300
 	-1   0    0    -1
