File: pcb/discrete/discrete-rf-board/lo.sch (KiCad schematic (older format))
At the start: 55 parts, among them J14 UFL, J15 UFL, Q14 BFU520R, U5 ADF4360-7BCPZRL7, U6 HHM17147A1, X1 ECS-5032MV-100-BN-TR

Commit message: Footprint a lot of stuff; save before autofill
Parts:
- C89: value 26.1 pF -> 27 pF; footprint (none) -> Capacitor_SMD:C_0402_1005Metric; Mouser (none) -> 80-C0402C270J5G
- C90: value 355 pF -> 360 pF; footprint (none) -> Capacitor_SMD:C_0402_1005Metric; Mouser (none) -> 963-UMK105CH361JVHF
- C96: footprint (none) -> Capacitor_SMD:C_0402_1005Metric; Mouser (none) -> 80-C0402C399C5HACTU
- L13: footprint (none) -> Capacitor_SMD:C_0402_1005Metric; Mouser (none) -> 81-LQG15HS3N9C02D
- R70: footprint (none) -> Resistor_SMD:R_0402_1005Metric; Mouser (none) -> 71-CRCW04023R30JNEDC
- R80: value 10R -> 22R
- R81: footprint (none) -> Resistor_SMD:R_0402_1005Metric; Mouser (none) -> 667-ERJ-U02D10R0X
Changed lines of the file:
@@
 F 0 "L13" H 1730 4640 50  0000 L CNN
 F 1 "3.9 nH" H 1730 4560 50  0000 L CNN
-F 2 "" H 1700 4600 50  0001 C CNN
+F 2 "Capacitor_SMD:C_0402_1005Metric" H 1700 4600 50  0001 C CNN
 F 3 "~" H 1700 4600 50  0001 C CNN
+F 4 "81-LQG15HS3N9C02D" H 1700 4600 50  0001 C CNN "Mouser"
 	1    1700 4600
 	-1   0    0    -1
@@
 F 0 "R70" H 4880 3070 50  0000 L CNN
 F 1 "3.3R" H 4880 3010 50  0000 L CNN
-F 2 "" H 4850 3050 50  0001 C CNN
+F 2 "Resistor_SMD:R_0402_1005Metric" H 4850 3050 50  0001 C CNN
 F 3 "~" H 4850 3050 50  0001 C CNN
+F 4 "71-CRCW04023R30JNEDC" H 4850 3050 50  0001 C CNN "Mouser"
 	1    4850 3050
 	1    0    0    -1
@@
 F 0 "C96" H 5810 3770 50  0000 L CNN
 F 1 "3.9 pF" H 5810 3620 50  0000 L CNN
-F 2 "" H 5800 3700 50  0001 C CNN
+F 2 "Capacitor_SMD:C_0402_1005Metric" H 5800 3700 50  0001 C CNN
 F 3 "~" H 5800 3700 50  0001 C CNN
+F 4 "80-C0402C399C5HACTU" H 5800 3700 50  0001 C CNN "Mouser"
 	1    5800 3700
 	0    -1   1    0
@@
 P 9450 3050
 F 0 "R80" H 9480 3070 50  0000 L CNN
-F 1 "10R" H 9480 3010 50  0000 L CNN
+F 1 "22R" H 9480 3010 50  0000 L CNN
 F 2 "" H 9450 3050 50  0001 C CNN
 F 3 "~" H 9450 3050 50  0001 C CNN
@@
 P 4850 4650
 F 0 "C89" H 4860 4720 50  0000 L CNN
-F 1 "26.1 pF" H 4860 4570 50  0000 L CNN
-F 2 "" H 4850 4650 50  0001 C CNN
+F 1 "27 pF" H 4860 4570 50  0000 L CNN
+F 2 "Capacitor_SMD:C_0402_1005Metric" H 4850 4650 50  0001 C CNN
 F 3 "~" H 4850 4650 50  0001 C CNN
+F 4 "80-C0402C270J5G" H 4850 4650 50  0001 C CNN "Mouser"
 	1    4850 4650
 	1    0    0    -1
@@
 P 5200 4950
 F 0 "C90" H 5210 5020 50  0000 L CNN
-F 1 "355 pF" H 5210 4870 50  0000 L CNN
-F 2 "" H 5200 4950 50  0001 C CNN
+F 1 "360 pF" H 5210 4870 50  0000 L CNN
+F 2 "Capacitor_SMD:C_0402_1005Metric" H 5200 4950 50  0001 C CNN
 F 3 "~" H 5200 4950 50  0001 C CNN
+F 4 "963-UMK105CH361JVHF" H 5200 4950 50  0001 C CNN "Mouser"
 	1    5200 4950
 	1    0    0    -1
@@
 F 0 "R81" H 9480 4720 50  0000 L CNN
 F 1 "10R" H 9480 4660 50  0000 L CNN
-F 2 "" H 9450 4700 50  0001 C CNN
+F 2 "Resistor_SMD:R_0402_1005Metric" H 9450 4700 50  0001 C CNN
 F 3 "~" H 9450 4700 50  0001 C CNN
+F 4 "667-ERJ-U02D10R0X" H 9450 4700 50  0001 C CNN "Mouser"
 	1    9450 4700
 	-1   0    0    -1

Commit message: Autofill
Parts:
- C107, C92, C95: footprint (none) -> Capacitor_SMD:C_0402_1005Metric; Mouser (none) -> 80-C0402C102K5R7411
- C99: footprint (none) -> Capacitor_SMD:C_0402_1005Metric; Mouser (none) -> 80-C0402C399C5HACTU
- L14: footprint (none) -> Capacitor_SMD:C_0402_1005Metric; Mouser (none) -> 81-LQG15HS3N9C02D
- L20: footprint (none) -> Capacitor_SMD:C_0402_1005Metric; Mouser (none) -> 963-HK1005R22J-T
- R73: footprint (none) -> Resistor_SMD:R_0402_1005Metric; Mouser (none) -> 71-CRCW04023R30JNEDC
- R79: footprint (none) -> Resistor_SMD:R_0402_1005Metric; Mouser (none) -> 667-ERJ-U02D10R0X
- R80: footprint (none) -> Resistor_SMD:R_0402_1005Metric; Mouser (none) -> 71-CRCW040222R0JNEDC
Changed lines of the file:
@@
 F 0 "L14" H 2130 4640 50  0000 L CNN
 F 1 "3.9 nH" H 2130 4560 50  0000 L CNN
-F 2 "" H 2100 4600 50  0001 C CNN
+F 2 "Capacitor_SMD:C_0402_1005Metric" H 2100 4600 50  0001 C CNN
 F 3 "~" H 2100 4600 50  0001 C CNN
+F 4 "81-LQG15HS3N9C02D" H 2100 4600 50  0001 C CNN "Mouser"
 	1    2100 4600
 	-1   0    0    -1
@@
 F 0 "C92" H 5410 3020 50  0000 L CNN
 F 1 "1 nF" H 5410 2870 50  0000 L CNN
-F 2 "" H 5400 2950 50  0001 C CNN
+F 2 "Capacitor_SMD:C_0402_1005Metric" H 5400 2950 50  0001 C CNN
 F 3 "~" H 5400 2950 50  0001 C CNN
+F 4 "80-C0402C102K5R7411" H 5400 2950 50  0001 C CNN "Mouser"
 	1    5400 2950
 	1    0    0    -1
@@
 F 0 "C95" H 5810 3020 50  0000 L CNN
 F 1 "1 nF" H 5810 2870 50  0000 L CNN
-F 2 "" H 5800 2950 50  0001 C CNN
+F 2 "Capacitor_SMD:C_0402_1005Metric" H 5800 2950 50  0001 C CNN
 F 3 "~" H 5800 2950 50  0001 C CNN
+F 4 "80-C0402C102K5R7411" H 5800 2950 50  0001 C CNN "Mouser"
 	1    5800 2950
 	1    0    0    -1
@@
 F 0 "R73" H 6480 2970 50  0000 L CNN
 F 1 "3.3R" H 6480 2910 50  0000 L CNN
-F 2 "" H 6450 2950 50  0001 C CNN
+F 2 "Resistor_SMD:R_0402_1005Metric" H 6450 2950 50  0001 C CNN
 F 3 "~" H 6450 2950 50  0001 C CNN
+F 4 "71-CRCW04023R30JNEDC" H 6450 2950 50  0001 C CNN "Mouser"
 	1    6450 2950
 	1    0    0    -1
@@
 F 0 "C99" H 6610 3770 50  0000 L CNN
 F 1 "3.9 pF" H 6610 3620 50  0000 L CNN
-F 2 "" H 6600 3700 50  0001 C CNN
+F 2 "Capacitor_SMD:C_0402_1005Metric" H 6600 3700 50  0001 C CNN
 F 3 "~" H 6600 3700 50  0001 C CNN
+F 4 "80-C0402C399C5HACTU" H 6600 3700 50  0001 C CNN "Mouser"
 	1    6600 3700
 	0    -1   1    0
@@
 F 0 "L20" H 9480 3590 50  0000 L CNN
 F 1 "220 nH" H 9480 3510 50  0000 L CNN
-F 2 "" H 9450 3550 50  0001 C CNN
+F 2 "Capacitor_SMD:C_0402_1005Metric" H 9450 3550 50  0001 C CNN
 F 3 "~" H 9450 3550 50  0001 C CNN
+F 4 "963-HK1005R22J-T" H 9450 3550 50  0001 C CNN "Mouser"
 	1    9450 3550
 	-1   0    0    -1
@@
 F 0 "R80" H 9480 3070 50  0000 L CNN
 F 1 "22R" H 9480 3010 50  0000 L CNN
-F 2 "" H 9450 3050 50  0001 C CNN
+F 2 "Resistor_SMD:R_0402_1005Metric" H 9450 3050 50  0001 C CNN
 F 3 "~" H 9450 3050 50  0001 C CNN
+F 4 "71-CRCW040222R0JNEDC" H 9450 3050 50  0001 C CNN "Mouser"
 	1    9450 3050
 	1    0    0    -1
@@
 F 0 "C107" H 10560 3070 50  0000 L CNN
 F 1 "1 nF" H 10560 2920 50  0000 L CNN
-F 2 "" H 10550 3000 50  0001 C CNN
+F 2 "Capacitor_SMD:C_0402_1005Metric" H 10550 3000 50  0001 C CNN
 F 3 "~" H 10550 3000 50  0001 C CNN
+F 4 "80-C0402C102K5R7411" H 10550 3000 50  0001 C CNN "Mouser"
 	1    10550 3000
 	1    0    0    -1
@@
 F 0 "R79" H 8880 4220 50  0000 L CNN
 F 1 "10R" H 8880 4160 50  0000 L CNN
-F 2 "" H 8850 4200 50  0001 C CNN
+F 2 "Resistor_SMD:R_0402_1005Metric" H 8850 4200 50  0001 C CNN
 F 3 "~" H 8850 4200 50  0001 C CNN
+F 4 "667-ERJ-U02D10R0X" H 8850 4200 50  0001 C CNN "Mouser"
 	1    8850 4200
 	0    -1   1    0

Commit message: Add in a couple more components, save before autofill
Parts:
- L17: footprint (none) -> Capacitor_SMD:C_0402_1005Metric; Mouser (none) -> 81-LQG15HZ47NJ02D
- R69: value 4.70kR -> 4k7R; footprint (none) -> Resistor_SMD:R_0402_1005Metric; Mouser (none) -> 603-AC0402FR-134K7L
- R72: value 25.6kR -> 22kR; footprint (none) -> Resistor_SMD:R_0805_2012Metric_Pad1.15x1.40mm_HandSolder; Mouser (none) -> 71-CRCW080522K0FKEAC
Changed lines of the file:
@@
 P 2950 5000
 F 0 "R69" H 2980 5020 50  0000 L CNN
-F 1 "4.70kR" H 2980 4960 50  0000 L CNN
-F 2 "" H 2950 5000 50  0001 C CNN
+F 1 "4k7R" H 2980 4960 50  0000 L CNN
+F 2 "Resistor_SMD:R_0402_1005Metric" H 2950 5000 50  0001 C CNN
 F 3 "~" H 2950 5000 50  0001 C CNN
+F 4 "603-AC0402FR-134K7L" H 2950 5000 50  0001 C CNN "Mouser"
 	1    2950 5000
 	-1   0    0    -1
@@
 F 0 "L17" H 6480 3540 50  0000 L CNN
 F 1 "47 nH" H 6480 3460 50  0000 L CNN
-F 2 "" H 6450 3500 50  0001 C CNN
+F 2 "Capacitor_SMD:C_0402_1005Metric" H 6450 3500 50  0001 C CNN
 F 3 "~" H 6450 3500 50  0001 C CNN
+F 4 "81-LQG15HZ47NJ02D" H 6450 3500 50  0001 C CNN "Mouser"
 	1    6450 3500
 	1    0    0    -1
@@
 P 5400 4400
 F 0 "R72" H 5430 4420 50  0000 L CNN
-F 1 "25.6kR" H 5430 4360 50  0000 L CNN
-F 2 "" H 5400 4400 50  0001 C CNN
+F 1 "22kR" H 5430 4360 50  0000 L CNN
+F 2 "Resistor_SMD:R_0805_2012Metric_Pad1.15x1.40mm_HandSolder" H 5400 4400 50  0001 C CNN
 F 3 "~" H 5400 4400 50  0001 C CNN
+F 4 "71-CRCW080522K0FKEAC" H 5400 4400 50  0001 C CNN "Mouser"
 	1    5400 4400
 	0    -1   -1   0

Commit message: Autofill
Parts:
- L15: footprint (none) -> Capacitor_SMD:C_0402_1005Metric; Mouser (none) -> 81-LQG15HZ47NJ02D
- L19, L21: footprint (none) -> Capacitor_SMD:C_0402_1005Metric; Mouser (none) -> NoPart
- R67, R68: footprint (none) -> Resistor_SMD:R_0402_1005Metric; Mouser (none) -> 603-RC0402JR-13470RL
- R75: footprint (none) -> Resistor_SMD:R_0402_1005Metric; Mouser (none) -> NoPart
Changed lines of the file:
@@
 F 0 "L15" H 5680 3540 50  0000 L CNN
 F 1 "47 nH" H 5680 3460 50  0000 L CNN
-F 2 "" H 5650 3500 50  0001 C CNN
+F 2 "Capacitor_SMD:C_0402_1005Metric" H 5650 3500 50  0001 C CNN
 F 3 "~" H 5650 3500 50  0001 C CNN
+F 4 "81-LQG15HZ47NJ02D" H 5650 3500 50  0001 C CNN "Mouser"
 	1    5650 3500
 	1    0    0    -1
@@
 F 0 "R67" H 1330 4620 50  0000 L CNN
 F 1 "470R" H 1330 4560 50  0000 L CNN
-F 2 "" H 1300 4600 50  0001 C CNN
+F 2 "Resistor_SMD:R_0402_1005Metric" H 1300 4600 50  0001 C CNN
 F 3 "~" H 1300 4600 50  0001 C CNN
+F 4 "603-RC0402JR-13470RL" H 1300 4600 50  0001 C CNN "Mouser"
 	1    1300 4600
 	-1   0    0    -1
@@
 F 0 "R68" H 2480 4620 50  0000 L CNN
 F 1 "470R" H 2480 4560 50  0000 L CNN
-F 2 "" H 2450 4600 50  0001 C CNN
+F 2 "Resistor_SMD:R_0402_1005Metric" H 2450 4600 50  0001 C CNN
 F 3 "~" H 2450 4600 50  0001 C CNN
+F 4 "603-RC0402JR-13470RL" H 2450 4600 50  0001 C CNN "Mouser"
 	1    2450 4600
 	-1   0    0    -1
@@
 F 0 "R75" H 7930 4470 50  0000 L CNN
 F 1 "DNP 0402" H 7930 4410 50  0000 L CNN
-F 2 "" H 7900 4450 50  0001 C CNN
+F 2 "Resistor_SMD:R_0402_1005Metric" H 7900 4450 50  0001 C CNN
 F 3 "~" H 7900 4450 50  0001 C CNN
+F 4 "NoPart" H 7900 4450 50  0001 C CNN "Mouser"
 	1    7900 4450
 	1    0    0    -1
@@
 F 0 "L19" H 8380 4490 50  0000 L CNN
 F 1 "TBD 0402" H 8380 4410 50  0000 L CNN
-F 2 "" H 8350 4450 50  0001 C CNN
+F 2 "Capacitor_SMD:C_0402_1005Metric" H 8350 4450 50  0001 C CNN
 F 3 "~" H 8350 4450 50  0001 C CNN
+F 4 "NoPart" H 8350 4450 50  0001 C CNN "Mouser"
 	1    8350 4450
 	1    0    0    -1
@@
 F 0 "L21" H 10180 4190 50  0000 L CNN
 F 1 "TBD 0402" H 10180 4110 50  0000 L CNN
-F 2 "" H 10150 4150 50  0001 C CNN
+F 2 "Capacitor_SMD:C_0402_1005Metric" H 10150 4150 50  0001 C CNN
 F 3 "~" H 10150 4150 50  0001 C CNN
+F 4 "NoPart" H 10150 4150 50  0001 C CNN "Mouser"
 	1    10150 4150
 	1    0    0    -1
