File: pcb/discrete/discrete-rf-board/mixer.sch (KiCad schematic (older format))
At the start: 50 parts, among them J7 UFL, J8 UFL, Q1 NSVT65011MW6T1G, Q2 BCM857BS-7-F, Q3 Q_NPN_BCE, Q4 BCM857BS-7-F, Q5 NSVT65011MW6T1G, T1 HHM1515B2, U3 LT5560EDD#PBF

Commit message: Autofill
Parts:
- R10, R16, R17: footprint (none) -> Resistor_SMD:R_0402_1005Metric; Mouser (none) -> 603-AC0402FR-134K7L
Changed lines of the file:
@@
 F 0 "R31" H 3430 5470 50  0000 L CNN
 F 1 "4k7R" H 3430 5410 50  0000 L CNN
-F 2 "" H 3400 5450 50  0001 C CNN
+F 2 "Resistor_SMD:R_0402_1005Metric" H 3400 5450 50  0001 C CNN
 F 3 "~" H 3400 5450 50  0001 C CNN
+F 4 "603-AC0402FR-134K7L" H 3400 5450 50  0001 C CNN "Mouser"
 	1    3400 5450
 	1    0    0    -1
@@
 F 0 "R24" H 1459 2296 50  0000 L CNN
 F 1 "4k7R" H 1459 2205 50  0000 L CNN
-F 2 "" H 1400 2250 50  0001 C CNN
+F 2 "Resistor_SMD:R_0402_1005Metric" H 1400 2250 50  0001 C CNN
 F 3 "~" H 1400 2250 50  0001 C CNN
+F 4 "603-AC0402FR-134K7L" H 1400 2250 50  0001 C CNN "Mouser"
 	1    1400 2250
 	1    0    0    -1
@@
 F 0 "R30" H 3259 2246 50  0000 L CNN
 F 1 "4k7R" H 3259 2155 50  0000 L CNN
-F 2 "" H 3200 2200 50  0001 C CNN
+F 2 "Resistor_SMD:R_0402_1005Metric" H 3200 2200 50  0001 C CNN
 F 3 "~" H 3200 2200 50  0001 C CNN
+F 4 "603-AC0402FR-134K7L" H 3200 2200 50  0001 C CNN "Mouser"
 	1    3200 2200
 	1    0    0    -1
