File: pcb/discrete/discrete-rf-board/transmitter.sch (KiCad schematic (older format))
At the start: 8 parts

Commit message: Reannotate everything; I'm trying to cut down the number of components
Connections:
- net at FL2.2 (SUM): now also FL3.1 (IN)
Changed lines of the file:
@@
 Connection ~ 6750 3350
 $Comp
-L power:GND #PWR026
+L power:GND #PWR022
 U 1 1 5D7F5C8F
 P 7550 4150
-F 0 "#PWR026" H 7550 3900 50  0001 C CNN
+F 0 "#PWR022" H 7550 3900 50  0001 C CNN
 F 1 "GND" H 7550 4000 50  0000 C CNN
 F 2 "" H 7550 4150 50  0001 C CNN
@@
 	1200 3700 1250 3700
 $Comp
-L power:GND #PWR020
+L power:GND #PWR016
 U 1 1 5D8C821A
 P 1200 4050
-F 0 "#PWR020" H 1200 3800 50  0001 C CNN
+F 0 "#PWR016" H 1200 3800 50  0001 C CNN
 F 1 "GND" H 1200 3900 50  0000 C CNN
 F 2 "" H 1200 4050 50  0001 C CNN
@@
 	1200 4050 1200 3950
 $Comp
-L power:GND #PWR021
+L power:GND #PWR017
 U 1 1 5D8C8A04
 P 1550 4050
-F 0 "#PWR021" H 1550 3800 50  0001 C CNN
+F 0 "#PWR017" H 1550 3800 50  0001 C CNN
 F 1 "GND" H 1550 3900 50  0000 C CNN
 F 2 "" H 1550 4050 50  0001 C CNN
@@
 	1550 4050 1550 3950
 $Comp
-L power:GND #PWR022
+L power:GND #PWR018
 U 1 1 5D8C95C0
 P 1950 4300
-F 0 "#PWR022" H 1950 4050 50  0001 C CNN
+F 0 "#PWR018" H 1950 4050 50  0001 C CNN
 F 1 "GND" H 1950 4150 50  0000 C CNN
 F 2 "" H 1950 4300 50  0001 C CNN
@@
 	1950 4300 1950 4200
 $Comp
-L power:GND #PWR023
+L power:GND #PWR019
 U 1 1 5D8CA782
 P 2500 4200
-F 0 "#PWR023" H 2500 3950 50  0001 C CNN
+F 0 "#PWR019" H 2500 3950 50  0001 C CNN
 F 1 "GND" H 2500 4050 50  0000 C CNN
 F 2 "" H 2500 4200 50  0001 C CNN
@@
 	7800 3550 8000 3550
 $Comp
-L power:GND #PWR027
+L power:GND #PWR023
 U 1 1 5DCABC6C
 P 8200 4050
-F 0 "#PWR027" H 8200 3800 50  0001 C CNN
+F 0 "#PWR023" H 8200 3800 50  0001 C CNN
 F 1 "GND" H 8200 3900 50  0000 C CNN
 F 2 "" H 8200 4050 50  0001 C CNN
@@
 $EndComp
 $Comp
-L power:GND #PWR028
+L power:GND #PWR024
 U 1 1 5DCABEC4
 P 8600 4050
-F 0 "#PWR028" H 8600 3800 50  0001 C CNN
+F 0 "#PWR024" H 8600 3800 50  0001 C CNN
 F 1 "GND" H 8600 3900 50  0000 C CNN
 F 2 "" H 8600 4050 50  0001 C CNN
@@
 PA_GND
 $Comp
-L power:GND #PWR029
+L power:GND #PWR025
 U 1 1 5D8EC555
 P 10400 2700
-F 0 "#PWR029" H 10400 2450 50  0001 C CNN
+F 0 "#PWR025" H 10400 2450 50  0001 C CNN
 F 1 "GND" H 10400 2550 50  0000 C CNN
 F 2 "" H 10400 2700 50  0001 C CNN
@@
 I_MIX_GND
 $Comp
-L power:GND #PWR025
+L power:GND #PWR021
 U 1 1 5D8EF6D5
 P 5800 1900
-F 0 "#PWR025" H 5800 1650 50  0001 C CNN
+F 0 "#PWR021" H 5800 1650 50  0001 C CNN
 F 1 "GND" H 5800 1750 50  0000 C CNN
 F 2 "" H 5800 1900 50  0001 C CNN
@@
 Q_MIX_GND
 $Comp
-L power:GND #PWR024
+L power:GND #PWR020
 U 1 1 5D8F1675
 P 5750 3600
-F 0 "#PWR024" H 5750 3350 50  0001 C CNN
+F 0 "#PWR020" H 5750 3350 50  0001 C CNN
 F 1 "GND" H 5750 3450 50  0000 C CNN
 F 2 "" H 5750 3600 50  0001 C CNN

Commit message: Footprint more stuff
Parts:
- R6: footprint (none) -> Resistor_SMD:R_0402_1005Metric; Mouser (none) -> 603-RC0402JR-0750RL
- R7: value 50R 0603 -> 51R 0603; footprint (none) -> Resistor_SMD:R_0603_1608Metric_Pad1.05x0.95mm_HandSolder; Mouser (none) -> 603-RC0603FR-0751RL
Connections:
- net at FL2.2 (SUM): now also FL3.1 (IN)
Changed lines of the file:
@@
 P 6750 3550
 F 0 "R7" H 6780 3570 50  0000 L CNN
-F 1 "50R 0603" H 6780 3510 50  0000 L CNN
-F 2 "" H 6750 3550 50  0001 C CNN
+F 1 "51R 0603" H 6780 3510 50  0000 L CNN
+F 2 "Resistor_SMD:R_0603_1608Metric_Pad1.05x0.95mm_HandSolder" H 6750 3550 50  0001 C CNN
 F 3 "~" H 6750 3550 50  0001 C CNN
+F 4 "603-RC0603FR-0751RL" H 6750 3550 50  0001 C CNN "Mouser"
 	1    6750 3550
 	1    0    0    -1
@@
 F 0 "R6" H 1980 4120 50  0000 L CNN
 F 1 "50R" H 1980 4060 50  0000 L CNN
-F 2 "" H 1950 4100 50  0001 C CNN
+F 2 "Resistor_SMD:R_0402_1005Metric" H 1950 4100 50  0001 C CNN
 F 3 "~" H 1950 4100 50  0001 C CNN
+F 4 "603-RC0402JR-0750RL" H 1950 4100 50  0001 C CNN "Mouser"
 	1    1950 4100
 	1    0    0    -1
