File: pcb/discrete/discrete-rf-board/dac.sch (KiCad schematic (older format))
At the start: 19 parts, among them Q12 Q_NPN_BCE

Commit message: Autofill
Parts:
- R53, R54: footprint (none) -> Resistor_SMD:R_0402_1005Metric; Mouser (none) -> 667-ERJ-2RKF7501X
Changed lines of the file:
@@
 F 0 "R53" H 3580 3320 50  0000 L CNN
 F 1 "7.5kR 1%" H 3580 3260 50  0000 L CNN
-F 2 "" H 3550 3300 50  0001 C CNN
+F 2 "Resistor_SMD:R_0402_1005Metric" H 3550 3300 50  0001 C CNN
 F 3 "~" H 3550 3300 50  0001 C CNN
+F 4 "667-ERJ-2RKF7501X" H 3550 3300 50  0001 C CNN "Mouser"
 	1    3550 3300
 	1    0    0    -1
@@
 F 0 "R54" H 3580 3620 50  0000 L CNN
 F 1 "7.5kR 1%" H 3580 3560 50  0000 L CNN
-F 2 "" H 3550 3600 50  0001 C CNN
+F 2 "Resistor_SMD:R_0402_1005Metric" H 3550 3600 50  0001 C CNN
 F 3 "~" H 3550 3600 50  0001 C CNN
+F 4 "667-ERJ-2RKF7501X" H 3550 3600 50  0001 C CNN "Mouser"
 	1    3550 3600
 	1    0    0    -1
