File: pcb/discrete/test-mixer/test-mixer/test-mixer.sch (KiCad schematic (older format))
At the start: 77 parts, among them J1 UFL, J2 UFL, J3 SMA, J4 Conn_01x08, J5 Conn_01x01, J6 Conn_01x01, T1 HHM17147A1, T2 HHM17147A1, U1 ADF4360-7BCPZ, U2 BAT15-099R, X1 EC5-5032MV-100-BN-TR

Commit message: Footprint everything(?)
Parts:
- C1: footprint (none) -> Capacitor_SMD:C_0603_1608Metric_Pad1.05x0.95mm_HandSolder; Mouser (none) -> 791-RF18N101J500CT
- C14: footprint (none) -> Capacitor_SMD:C_0402_1005Metric; Mouser (none) -> 81-GJM1555C1H3R9CB1D
- C18: footprint (none) -> Capacitor_SMD:C_0603_1608Metric_Pad1.05x0.95mm_HandSolder; Mouser (none) -> 80-C0603C270K5G
- C19: footprint (none) -> Capacitor_SMD:C_0805_2012Metric_Pad1.15x1.40mm_HandSolder; Mouser (none) -> 80-C0805C120J1HACTU
- C20: footprint (none) -> Capacitor_SMD:C_0402_1005Metric; Mouser (none) -> 963-UMK105CH361JVHF
- C22: footprint (none) -> Capacitor_SMD:C_0805_2012Metric_Pad1.15x1.40mm_HandSolder; Mouser (none) -> 81-GRM21BC81C106KE5L
- C5: footprint (none) -> Capacitor_SMD:C_0402_1005Metric; Mouser (none) -> 80-C0402C103K4R7411
- C7: footprint (none) -> Capacitor_SMD:C_0402_1005Metric; Mouser (none) -> 80-C0402C104M4P
- J1: footprint (none) -> discrete_footprints:2337019-1; Mouser (none) -> 571-2337019-1
- J3: footprint (none) -> discrete_footprints:142-0701-801-with-taper; Mouser (none) -> 530-142-0701-801
- J4: footprint (none) -> Connector_PinHeader_2.54mm:PinHeader_1x08_P2.54mm_Vertical; Mouser (none) -> NoPart
- J5: footprint (none) -> Connector_PinSocket_2.54mm:PinSocket_1x01_P2.54mm_Vertical; Mouser (none) -> NoPart
- L1: footprint (none) -> Capacitor_SMD:C_0402_1005Metric; Mouser (none) -> 81-LQG15HZ47NJ02D
- L16: footprint (none) -> Capacitor_SMD:C_0402_1005Metric; Mouser (none) -> 81-LQG15HS3N9C02D
- L3: footprint (none) -> Capacitor_SMD:C_0402_1005Metric; Mouser (none) -> 81-LQG15HN7N5J02D
- R1: footprint (none) -> Resistor_SMD:R_0603_1608Metric_Pad1.05x0.95mm_HandSolder; Mouser (none) -> 652-CR0603-J/-3R3ELF
- R13: footprint (none) -> Resistor_SMD:R_0603_1608Metric_Pad1.05x0.95mm_HandSolder; Mouser (none) -> 603-RC0603FR-1027KL
- R14: footprint (none) -> Resistor_SMD:R_0603_1608Metric_Pad1.05x0.95mm_HandSolder; Mouser (none) -> 652-CR0603FX-1202ELF
- R18: footprint (none) -> Resistor_SMD:R_0402_1005Metric; Mouser (none) -> 603-AC0402FR-134K7L
- R3: footprint (none) -> Resistor_SMD:R_0402_1005Metric; Mouser (none) -> 71-CRCW04020000Z0EDC
- R4: footprint (none) -> Resistor_SMD:R_0402_1005Metric; Mouser (none) -> 603-RC0402JR-13470RL
- TP2: footprint (none) -> TestPoint:TestPoint_Pad_D1.0mm; Mouser (none) -> NoPart
- U1: footprint (none) -> discrete_footprints:Analog_CP-24-14
- U2: footprint (none) -> discrete_footprints:NXP_SOT143B
- X1: footprint Oscillator:Oscillator_SMD_ECS_2520MV-xxx-xx-4Pin_2.5x2.0mm -> Oscillator:Oscillator_SMD_SeikoEpson_SG8002LB-4Pin_5.0x3.2mm_HandSoldering
Changed lines of the file:
@@
 F 0 "U1" H 3500 4300 50  0000 C CNN
 F 1 "ADF4360-7BCPZ" H 3500 4150 50  0000 C CNN
-F 2 "" H 3500 3850 50  0001 C CNN
+F 2 "discrete_footprints:Analog_CP-24-14" H 3500 3850 50  0001 C CNN
 F 3 "" H 3500 3850 50  0001 C CNN
 F 4 "584-ADF4360-7BCPZR7" H 3500 3850 50  0000 C CNN "Mouser"
@@
 F 0 "U2" H 8050 4200 50  0000 C CNN
 F 1 "BAT15-099R" H 8050 3600 50  0000 C CNN
-F 2 "" H 8050 4200 50  0001 C CNN
+F 2 "discrete_footprints:NXP_SOT143B" H 8050 4200 50  0001 C CNN
 F 3 "" H 8050 4200 50  0001 C CNN
 F 4 "726-BAT15099RE6327" H 8050 3500 50  0000 C CNN "Mouser"
@@
 F 0 "J3" H 10310 3870 50  0000 C CNN
 F 1 "SMA" V 10415 3750 50  0000 C CNN
-F 2 "" H 10300 3750 50  0001 C CNN
+F 2 "discrete_footprints:142-0701-801-with-taper" H 10300 3750 50  0001 C CNN
 F 3 " ~" H 10300 3750 50  0001 C CNN
+F 4 " 530-142-0701-801 " H 10300 3750 50  0001 C CNN "Mouser"
 	1    10300 3750
 	1    0    0    -1
@@
 F 0 "J1" H 6660 3870 50  0000 C CNN
 F 1 "UFL" V 6765 3750 50  0000 C CNN
-F 2 "" H 6650 3750 50  0001 C CNN
+F 2 "discrete_footprints:2337019-1" H 6650 3750 50  0001 C CNN
 F 3 " ~" H 6650 3750 50  0001 C CNN
+F 4 "571-2337019-1" H 6650 3750 50  0001 C CNN "Mouser"
 	1    6650 3750
 	-1   0    0    -1
@@
 F 0 "C14" H 5260 3820 50  0000 L CNN
 F 1 "3.9 pF" H 5260 3670 50  0000 L CNN
-F 2 "" H 5250 3750 50  0001 C CNN
+F 2 "Capacitor_SMD:C_0402_1005Metric" H 5250 3750 50  0001 C CNN
 F 3 "~" H 5250 3750 50  0001 C CNN
+F 4 "81-GJM1555C1H3R9CB1D" H 5250 3750 50  0001 C CNN "Mouser"
 	1    5250 3750
 	0    -1   1    0
@@
 F 0 "L3" H 5530 3790 50  0000 L CNN
 F 1 "7.5 nH" H 5530 3710 50  0000 L CNN
-F 2 "" H 5500 3750 50  0001 C CNN
+F 2 "Capacitor_SMD:C_0402_1005Metric" H 5500 3750 50  0001 C CNN
 F 3 "~" H 5500 3750 50  0001 C CNN
+F 4 "81-LQG15HN7N5J02D" H 5500 3750 50  0001 C CNN "Mouser"
 	1    5500 3750
 	0    -1   1    0
@@
 F 0 "L1" H 4780 3440 50  0000 L CNN
 F 1 "47 nH" H 4780 3360 50  0000 L CNN
-F 2 "" H 4750 3400 50  0001 C CNN
+F 2 "Capacitor_SMD:C_0402_1005Metric" H 4750 3400 50  0001 C CNN
 F 3 "~" H 4750 3400 50  0001 C CNN
+F 4 "81-LQG15HZ47NJ02D" H 4750 3400 50  0001 C CNN "Mouser"
 	1    4750 3400
 	1    0    0    -1
@@
 F 0 "J5" H 7750 4650 50  0000 C CNN
 F 1 "Conn_01x01" H 7750 4450 50  0000 C CNN
-F 2 "" H 7750 4550 50  0001 C CNN
+F 2 "Connector_PinSocket_2.54mm:PinSocket_1x01_P2.54mm_Vertical" H 7750 4550 50  0001 C CNN
 F 3 "~" H 7750 4550 50  0001 C CNN
+F 4 "NoPart" H 7750 4550 50  0001 C CNN "Mouser"
 	1    7750 4550
 	1    0    0    1
@@
 F 0 "C18" H 4460 4970 50  0000 L CNN
 F 1 "27 pF" H 4460 4820 50  0000 L CNN
-F 2 "" H 4450 4900 50  0001 C CNN
+F 2 "Capacitor_SMD:C_0603_1608Metric_Pad1.05x0.95mm_HandSolder" H 4450 4900 50  0001 C CNN
 F 3 "~" H 4450 4900 50  0001 C CNN
+F 4 "80-C0603C270K5G" H 4450 4900 50  0001 C CNN "Mouser"
 	1    4450 4900
 	1    0    0    -1
@@
 F 0 "C20" H 4910 5270 50  0000 L CNN
 F 1 "360 pF" H 4910 5120 50  0000 L CNN
-F 2 "" H 4900 5200 50  0001 C CNN
+F 2 "Capacitor_SMD:C_0402_1005Metric" H 4900 5200 50  0001 C CNN
 F 3 "~" H 4900 5200 50  0001 C CNN
+F 4 "963-UMK105CH361JVHF" H 4900 5200 50  0001 C CNN "Mouser"
 	1    4900 5200
 	1    0    0    -1
@@
 F 0 "R14" H 4930 4920 50  0000 L CNN
 F 1 "12k R" H 4930 4860 50  0000 L CNN
-F 2 "" H 4900 4900 50  0001 C CNN
+F 2 "Resistor_SMD:R_0603_1608Metric_Pad1.05x0.95mm_HandSolder" H 4900 4900 50  0001 C CNN
 F 3 "~" H 4900 4900 50  0001 C CNN
+F 4 "652-CR0603FX-1202ELF" H 4900 4900 50  0001 C CNN "Mouser"
 	1    4900 4900
 	1    0    0    -1
@@
 F 0 "R13" H 5180 4720 50  0000 L CNN
 F 1 "27k R" H 5180 4660 50  0000 L CNN
-F 2 "" H 5150 4700 50  0001 C CNN
+F 2 "Resistor_SMD:R_0603_1608Metric_Pad1.05x0.95mm_HandSolder" H 5150 4700 50  0001 C CNN
 F 3 "~" H 5150 4700 50  0001 C CNN
+F 4 "603-RC0603FR-1027KL" H 5150 4700 50  0001 C CNN "Mouser"
 	1    5150 4700
 	0    -1   -1   0
@@
 F 0 "C19" H 5360 4970 50  0000 L CNN
 F 1 "12 pF" H 5360 4820 50  0000 L CNN
-F 2 "" H 5350 4900 50  0001 C CNN
+F 2 "Capacitor_SMD:C_0805_2012Metric_Pad1.15x1.40mm_HandSolder" H 5350 4900 50  0001 C CNN
 F 3 "~" H 5350 4900 50  0001 C CNN
+F 4 "80-C0805C120J1HACTU" H 5350 4900 50  0001 C CNN "Mouser"
 	1    5350 4900
 	1    0    0    -1
@@
 F 0 "C22" H 2610 5320 50  0000 L CNN
 F 1 "10 uF" H 2610 5170 50  0000 L CNN
-F 2 "" H 2600 5250 50  0001 C CNN
+F 2 "Capacitor_SMD:C_0805_2012Metric_Pad1.15x1.40mm_HandSolder" H 2600 5250 50  0001 C CNN
 F 3 "~" H 2600 5250 50  0001 C CNN
+F 4 "81-GRM21BC81C106KE5L" H 2600 5250 50  0001 C CNN "Mouser"
 	1    2600 5250
 	1    0    0    -1
@@
 F 0 "R1" H 4380 1870 50  0000 L CNN
 F 1 "3.3 R" H 4380 1810 50  0000 L CNN
-F 2 "" H 4350 1850 50  0001 C CNN
+F 2 "Resistor_SMD:R_0603_1608Metric_Pad1.05x0.95mm_HandSolder" H 4350 1850 50  0001 C CNN
 F 3 "~" H 4350 1850 50  0001 C CNN
+F 4 "652-CR0603-J/-3R3ELF" H 4350 1850 50  0001 C CNN "Mouser"
 	1    4350 1850
 	1    0    0    -1
@@
 F 0 "C1" H 4610 2370 50  0000 L CNN
 F 1 "100 pF" H 4610 2220 50  0000 L CNN
-F 2 "" H 4600 2300 50  0001 C CNN
+F 2 "Capacitor_SMD:C_0603_1608Metric_Pad1.05x0.95mm_HandSolder" H 4600 2300 50  0001 C CNN
 F 3 "~" H 4600 2300 50  0001 C CNN
+F 4 "791-RF18N101J500CT" H 4600 2300 50  0001 C CNN "Mouser"
 	1    4600 2300
 	1    0    0    -1
@@
 F 0 "C5" H 6060 2370 50  0000 L CNN
 F 1 "10 nF" H 6060 2220 50  0000 L CNN
-F 2 "" H 6050 2300 50  0001 C CNN
+F 2 "Capacitor_SMD:C_0402_1005Metric" H 6050 2300 50  0001 C CNN
 F 3 "~" H 6050 2300 50  0001 C CNN
+F 4 " 80-C0402C103K4R7411 " H 6050 2300 50  0001 C CNN "Mouser"
 	1    6050 2300
 	1    0    0    -1
@@
 F 0 "R18" H 2280 5270 50  0000 L CNN
 F 1 "4k7 R" H 2280 5210 50  0000 L CNN
-F 2 "" H 2250 5250 50  0001 C CNN
+F 2 "Resistor_SMD:R_0402_1005Metric" H 2250 5250 50  0001 C CNN
 F 3 "~" H 2250 5250 50  0001 C CNN
+F 4 "603-AC0402FR-134K7L" H 2250 5250 50  0001 C CNN "Mouser"
 	1    2250 5250
 	1    0    0    -1
@@
 F 0 "L16" H 980 5040 50  0000 L CNN
 F 1 "3.9 nH" H 980 4960 50  0000 L CNN
-F 2 "" H 950 5000 50  0001 C CNN
+F 2 "Capacitor_SMD:C_0402_1005Metric" H 950 5000 50  0001 C CNN
 F 3 "~" H 950 5000 50  0001 C CNN
+F 4 "81-LQG15HS3N9C02D" H 950 5000 50  0001 C CNN "Mouser"
 	1    950  5000
 	1    0    0    -1
@@
 F 0 "R4" H 1280 3920 50  0000 L CNN
 F 1 "470 R" H 1280 3860 50  0000 L CNN
-F 2 "" H 1250 3900 50  0001 C CNN
+F 2 "Resistor_SMD:R_0402_1005Metric" H 1250 3900 50  0001 C CNN
 F 3 "~" H 1250 3900 50  0001 C CNN
+F 4 "603-RC0402JR-13470RL" H 1250 3900 50  0001 C CNN "Mouser"
 	1    1250 3900
 	0    -1   1    0
@@
 F 0 "X1" H 1250 3200 50  0000 L CNN
 F 1 "EC5-5032MV-100-BN-TR" H 1500 2700 50  0000 L CNN
-F 2 "Oscillator:Oscillator_SMD_ECS_2520MV-xxx-xx-4Pin_2.5x2.0mm" H 1900 2600 50  0001 C CNN
+F 2 "Oscillator:Oscillator_SMD_SeikoEpson_SG8002LB-4Pin_5.0x3.2mm_HandSoldering" H 1900 2600 50  0001 C CNN
 F 3 "https://www.ecsxtal.com/store/pdf/ECS-2520MV.pdf" H 1275 3075 50  0001 C CNN
 	1    1450 2950
@@
 F 0 "C7" H 1960 2670 50  0000 L CNN
 F 1 "0.1 uF" H 1960 2520 50  0000 L CNN
-F 2 "" H 1950 2600 50  0001 C CNN
+F 2 "Capacitor_SMD:C_0402_1005Metric" H 1950 2600 50  0001 C CNN
 F 3 "~" H 1950 2600 50  0001 C CNN
+F 4 "80-C0402C104M4P" H 1950 2600 50  0001 C CNN "Mouser"
 	1    1950 2600
 	1    0    0    -1
@@
 F 0 "TP2" H 1850 3920 50  0000 C CNN
 F 1 "-" H 1850 3850 50  0000 C CNN
-F 2 "" H 2050 3650 50  0001 C CNN
+F 2 "TestPoint:TestPoint_Pad_D1.0mm" H 2050 3650 50  0001 C CNN
 F 3 "~" H 2050 3650 50  0001 C CNN
+F 4 "NoPart" H 1850 3650 50  0001 C CNN "Mouser"
 	1    1850 3650
 	1    0    0    -1
@@
 F 0 "R3" H 6480 3570 50  0000 L CNN
 F 1 "0 R" H 6480 3510 50  0000 L CNN
-F 2 "" H 6450 3550 50  0001 C CNN
+F 2 "Resistor_SMD:R_0402_1005Metric" H 6450 3550 50  0001 C CNN
 F 3 "~" H 6450 3550 50  0001 C CNN
+F 4 "71-CRCW04020000Z0EDC" H 6450 3550 50  0001 C CNN "Mouser"
 	1    6450 3550
 	0    1    1    0
@@
 F 0 "J4" H 750 4400 50  0000 C CNN
 F 1 "Conn_01x08" H 750 3500 50  0000 C CNN
-F 2 "" H 750 4000 50  0001 C CNN
+F 2 "Connector_PinHeader_2.54mm:PinHeader_1x08_P2.54mm_Vertical" H 750 4000 50  0001 C CNN
 F 3 "~" H 750 4000 50  0001 C CNN
+F 4 "NoPart" H 750 4000 50  0001 C CNN "Mouser"
 	1    750  4000
 	-1   0    0    -1
