File: pcb/discrete/test-mixer/test-mixer.kicad_pcb (KiCad board)
At the start: 2 copper layers, 0 parts

Commit message: Finish layout
Parts:
- added C1: 100 pF, Capacitor_SMD:C_0603_1608Metric_Pad1.05x0.95mm_HandSolder, F.Cu at (38.5, 93.8)
- added C10: 100 pF, Capacitor_SMD:C_0603_1608Metric_Pad1.05x0.95mm_HandSolder, F.Cu at (45.4, 93.2)
- added C11: 100 pF, Capacitor_SMD:C_0603_1608Metric_Pad1.05x0.95mm_HandSolder, F.Cu at (45.4, 94.8)
- added C12: 10 nF, Capacitor_SMD:C_0402_1005Metric, F.Cu at (45.2, 96.2)
- added C13: 10 nF, Capacitor_SMD:C_0402_1005Metric, F.Cu at (45.2, 97.2)
- added C14: 3.9 pF, Capacitor_SMD:C_0402_1005Metric, F.Cu at (41.1, 96.7)
- added C15: TBD, Capacitor_SMD:C_0402_1005Metric, F.Cu at (41.2, 110.2)
- added C16: TBD, Capacitor_SMD:C_0402_1005Metric, F.Cu at (41.2, 118.7)
- added C17: 3.9 pF, Capacitor_SMD:C_0402_1005Metric, F.Cu at (42.1, 96.7)
- added C18: 27 pF, Capacitor_SMD:C_0603_1608Metric_Pad1.05x0.95mm_HandSolder, F.Cu at (33.5, 92.7)
- added C19: 12 pF, Capacitor_SMD:C_0805_2012Metric_Pad1.15x1.40mm_HandSolder, F.Cu at (49.1, 92.8)
- added C2: 100 pF, Capacitor_SMD:C_0603_1608Metric_Pad1.05x0.95mm_HandSolder, F.Cu at (37.2, 95.0)
- added C20: 360 pF, Capacitor_SMD:C_0402_1005Metric, F.Cu at (31.1, 93.5)
- added C21: 10 nF, Capacitor_SMD:C_0402_1005Metric, F.Cu at (44.7, 87.6)
- added C22: 10 uF, Capacitor_SMD:C_0805_2012Metric_Pad1.15x1.40mm_HandSolder, F.Cu at (42.0, 84.8)
- added C3: 100 pF, Capacitor_SMD:C_0603_1608Metric_Pad1.05x0.95mm_HandSolder, F.Cu at (34.8, 97.3)
- added C4: 100 pF, Capacitor_SMD:C_0603_1608Metric_Pad1.05x0.95mm_HandSolder, F.Cu at (33.4, 98.5)
- added C5: 10 nF, Capacitor_SMD:C_0402_1005Metric, F.Cu at (31.2, 100.2)
- added C6: 10 nF, Capacitor_SMD:C_0402_1005Metric, F.Cu at (32.1, 99.4)
- added C7: 0.1 uF, Capacitor_SMD:C_0402_1005Metric, F.Cu at (37.6, 78.3)
- added C8: 0.1 uF, Capacitor_SMD:C_0402_1005Metric, F.Cu at (37.5, 89.8)
- added C9: 0.1 uF, Capacitor_SMD:C_0402_1005Metric, F.Cu at (36.3, 89.9)
- added H1: MountingHole_Pad, MountingHole:MountingHole_3.2mm_M3_DIN965, F.Cu at (51.0, 80.0)
- added H2: MountingHole_Pad, MountingHole:MountingHole_3.2mm_M3_DIN965, F.Cu at (51.0, 137.0)
- added H3: MountingHole_Pad, MountingHole:MountingHole_3.2mm_M3_DIN965, F.Cu at (21.0, 137.0)
- added H4: MountingHole_Pad, MountingHole:MountingHole_3.2mm_M3_DIN965, F.Cu at (21.4, 105.8)
- added J1: UFL, discrete_footprints:2337019-1, F.Cu at (40.5, 105.4)
- added J2: UFL, discrete_footprints:2337019-1, F.Cu at (40.5, 124.5)
- added J3: SMA, discrete_footprints:142-0701-801-with-taper, F.Cu at (42.0, 141.2)
- added J4: Conn_01x08, Connector_PinHeader_2.54mm:PinHeader_1x08_P2.54mm_Vertical, F.Cu at (19.9, 79.1)
- added J5: Conn_01x01, Connector_PinSocket_2.54mm:PinSocket_1x01_P2.54mm_Vertical, F.Cu at (50.1, 110.8)
- added J6: Conn_01x01, Connector_PinSocket_2.54mm:PinSocket_1x01_P2.54mm_Vertical, F.Cu at (50.0, 118.5)
- added L1: 47 nH, Capacitor_SMD:C_0402_1005Metric, F.Cu at (41.1, 94.6)
- added L10: TBD, Capacitor_SMD:C_0402_1005Metric, F.Cu at (41.7, 111.8)
- added L11: TBD, Capacitor_SMD:C_0402_1005Metric, F.Cu at (41.7, 117.2)
- added L12: TBD, Capacitor_SMD:C_0402_1005Metric, F.Cu at (41.7, 120.2)
- added L13: 1 uH, Capacitor_SMD:C_0402_1005Metric, F.Cu at (45.0, 127.5)
- added L14: 1 uH, Capacitor_SMD:C_0402_1005Metric, F.Cu at (39.4, 102.8)
- added L15: 1 uH, Capacitor_SMD:C_0402_1005Metric, F.Cu at (42.8, 102.7)
- added L16: 3.9 nH, Capacitor_SMD:C_0402_1005Metric, F.Cu at (44.7, 91.2)
- added L17: 3.9 nH, Capacitor_SMD:C_0402_1005Metric, F.Cu at (45.9, 88.8)
- added L2: 47 nH, Capacitor_SMD:C_0402_1005Metric, F.Cu at (42.1, 94.6)
- added L3: 7.5 nH, Capacitor_SMD:C_0402_1005Metric, F.Cu at (41.1, 98.6)
- added L4: TBD, Capacitor_SMD:C_0402_1005Metric, F.Cu at (40.7, 108.7)
- added L5: TBD, Capacitor_SMD:C_0402_1005Metric, F.Cu at (40.7, 111.8)
- added L6: TBD, Capacitor_SMD:C_0402_1005Metric, F.Cu at (40.8, 117.2)
- added L7: TBD, Capacitor_SMD:C_0402_1005Metric, F.Cu at (40.8, 120.2)
- added L8: 7.5 nH, Capacitor_SMD:C_0402_1005Metric, F.Cu at (42.1, 98.6)
- added L9: TBD, Capacitor_SMD:C_0402_1005Metric, F.Cu at (41.7, 108.7)
- added R1: 3.3 R, Resistor_SMD:R_0603_1608Metric_Pad1.05x0.95mm_HandSolder, F.Cu at (28.5, 99.7)
- added R10: 470 R, Resistor_SMD:R_0402_1005Metric, F.Cu at (26.8, 91.0)
- added R11: TBD, Resistor_SMD:R_0402_1005Metric, F.Cu at (45.8, 111.3)
- added R12: TBD, Resistor_SMD:R_0402_1005Metric, F.Cu at (45.9, 117.1)
- added R13: 27k R, Resistor_SMD:R_0603_1608Metric_Pad1.05x0.95mm_HandSolder, F.Cu at (49.2, 94.6)
- added R14: 12k R, Resistor_SMD:R_0603_1608Metric_Pad1.05x0.95mm_HandSolder, F.Cu at (33.5, 94.3)
- added R15: TBD, Resistor_SMD:R_0402_1005Metric, F.Cu at (45.6, 114.2)
- added R16: 470 R, Resistor_SMD:R_0402_1005Metric, F.Cu at (45.7, 91.2)
- added R17: 470 R, Resistor_SMD:R_0402_1005Metric, F.Cu at (45.9, 89.7)
- added R18: 4k7 R, Resistor_SMD:R_0402_1005Metric, F.Cu at (43.6, 84.9)
- added R2: 3.3 R, Resistor_SMD:R_0603_1608Metric_Pad1.05x0.95mm_HandSolder, F.Cu at (45.2, 98.7)
- added R3: 0 R, Resistor_SMD:R_0402_1005Metric, F.Cu at (40.5, 102.7)
- added R4: 470 R, Resistor_SMD:R_0402_1005Metric, F.Cu at (26.8, 86.2)
- added R5: TBD, Resistor_SMD:R_0402_1005Metric, F.Cu at (41.2, 121.7)
- added R6: 470 R, Resistor_SMD:R_0402_1005Metric, F.Cu at (26.8, 87.3)
- added R7: 0 R, Resistor_SMD:R_0402_1005Metric, F.Cu at (41.6, 102.7)
- added R8: 470 R, Resistor_SMD:R_0402_1005Metric, F.Cu at (26.8, 88.5)
- added R9: 470 R, Resistor_SMD:R_0402_1005Metric, F.Cu at (26.8, 89.7)
- added T1: HHM17147A1, discrete_footprints:TDK_HHM17147A1, F.Cu at (41.5, 100.7)
- added T2: HHM17147A1, discrete_footprints:TDK_HHM17147A1, F.Cu at (41.4, 127.5)
- added TP1: -, TestPoint:TestPoint_Pad_D1.0mm, F.Cu at (40.0, 85.8)
- added TP2: -, TestPoint:TestPoint_Pad_D1.0mm, F.Cu at (29.8, 85.0)
- added TP3: -, TestPoint:TestPoint_Pad_D1.0mm, F.Cu at (29.9, 88.5)
- added TP4: -, TestPoint:TestPoint_Pad_D1.0mm, F.Cu at (30.1, 91.3)
- added TP5: -, TestPoint:TestPoint_Pad_D1.0mm, F.Cu at (31.9, 86.7)
- added TP6: -, TestPoint:TestPoint_Pad_D1.0mm, F.Cu at (31.9, 90.0)
- added TP7: -, TestPoint:TestPoint_Pad_D1.0mm, F.Cu at (50.2, 96.7)
- added TP8: -, TestPoint:TestPoint_Pad_D1.0mm, F.Cu at (45.8, 124.3)
- added TP9: -, TestPoint:TestPoint_Pad_D1.0mm, F.Cu at (45.9, 106.7)
- added U1: ADF4360-7BCPZ, discrete_footprints:Analog_CP-24-14, F.Cu at (41.1, 89.9)
- added U2: BAT15-099R, discrete_footprints:NXP_SOT143B, F.Cu at (41.2, 114.5)
- added X1: ECS-5032MV-100-BN-TR, Oscillator:Oscillator_SMD_SeikoEpson_SG8002LB-4Pin_5.0x3.2mm_HandSoldering, F.Cu at (37.8, 81.8)
Routing:
- net GND: track 0.00 -> 134.8 mm, vias 0 -> 82
- net /+3V3: track 0.00 -> 101.9 mm, vias 0 -> 2
- net /VVCO_3V3: track 0.00 -> 23.7 mm, vias 0 -> 3
- net Net-(L14-Pad2): track 0.00 -> 20.5 mm, vias 0 -> 2
- net Net-(C18-Pad1): track 0.00 -> 20.0 mm, vias 0 -> 2
- net Net-(C1-Pad1): track 0.00 -> 16.7 mm
- net Net-(R4-Pad2): track 0.00 -> 15.2 mm
- net Net-(L13-Pad2): track 0.00 -> 13.7 mm
- net Net-(R6-Pad2): track 0.00 -> 13.5 mm
- net Net-(R9-Pad2): track 0.00 -> 12.9 mm
- net Net-(R8-Pad2): track 0.00 -> 12.6 mm
- net Net-(R10-Pad2): track 0.00 -> 12.4 mm
- net Net-(C19-Pad1): track 0.00 -> 10.7 mm
- net /RF: track 0.00 -> 10.6 mm
- net Net-(J4-Pad7): track 0.00 -> 7.75 mm
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- added copper zone on F.Cu, net /+3V3
- added copper zone on B.Cu, net GND
- added copper zone on F.Cu, net GND
Other:
- board outline added: 38 x 65 mm
- net class Default: clearance 0.1524 -> 0.127
- rule trace_clearance: 0.1524 -> 0.127
- board text added: "Mixer test design Rev 1"
